File: HW/Camera.kicad_sch (KiCad schematic)
At the start: 0 parts

Commit message: Create probe pcb
Parts:
- added Camera: Conn_01x08, Connector_PinHeader_2.54mm:PinHeader_1x08_P2.54mm_Vertical, symbol Connector_Generic:Conn_01x08
Connections:
- new net 5V: Camera.6 (Pin_6)
- new net CAM_CS: Camera.1 (Pin_1)
- new net CAM_MISO: Camera.3 (Pin_3)
- new net CAM_MOSI: Camera.2 (Pin_2)
- new net CAM_SCK: Camera.4 (Pin_4)
- new net GND: Camera.5 (Pin_5)
- new net SCL: Camera.8 (Pin_8)
- new net SDA: Camera.7 (Pin_7)
Changed lines of the file:
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@@
 (kicad_sch (version 20230121) (generator eeschema)
   (paper "A4")
+  (wire (pts (xy 135.89 91.44) (xy 138.43 91.44))
+    (stroke (width 0) (type default))
+  )
+  (wire (pts (xy 135.89 86.36) (xy 138.43 86.36))
+    (stroke (width 0) (type default))
+  )
+  (wire (pts (xy 135.89 104.14) (xy 138.43 104.14))
+    (stroke (width 0) (type default))
+  )
+  (wire (pts (xy 135.89 101.6) (xy 138.43 101.6))
+    (stroke (width 0) (type default))
+  )
+  (wire (pts (xy 135.89 96.52) (xy 138.43 96.52))
+    (stroke (width 0) (type default))
+  )
+  (wire (pts (xy 135.89 99.06) (xy 138.43 99.06))
+    (stroke (width 0) (type default))
+  )
+  (wire (pts (xy 135.89 88.9) (xy 138.43 88.9))
+    (stroke (width 0) (type default))
+  )
+  (wire (pts (xy 135.89 93.98) (xy 138.43 93.98))
+    (stroke (width 0) (type default))
+  )
+  (global_label "CAM_SCK" (shape input) (at 135.89 93.98 180) (fields_autoplaced)
+    (effects (font (size 1.27 1.27)) (justify right))
+    (property "Intersheetrefs" "${INTERSHEET_REFS}" (at 124.4571 93.98 0)
+      (effects (font (size 1.27 1.27)) (justify right) hide)
+    )
+  )
+  (global_label "CAM_CS" (shape input) (at 135.89 86.36 180) (fields_autoplaced)
+    (effects (font (size 1.27 1.27)) (justify right))
+    (property "Intersheetrefs" "${INTERSHEET_REFS}" (at 125.7271 86.36 0)
+      (effects (font (size 1.27 1.27)) (justify right) hide)
+    )
+  )
+  (global_label "5V" (shape input) (at 135.89 99.06 180) (fields_autoplaced)
+    (effects (font (size 1.27 1.27)) (justify right))
+    (property "Intersheetrefs" "${INTERSHEET_REFS}" (at 130.6861 99.06 0)
+      (effects (font (size 1.27 1.27)) (justify right) hide)
+    )
+  )
+  (global_label "CAM_MOSI" (shape input) (at 135.89 88.9 180) (fields_autoplaced)
+    (effects (font (size 1.27 1.27)) (justify right))
+    (property "Intersheetrefs" "${INTERSHEET_REFS}" (at 123.6104 88.9 0)
+      (effects (font (size 1.27 1.27)) (justify right) hide)
+    )
+  )
+  (global_label "CAM_MISO" (shape input) (at 135.89 91.44 180) (fields_autoplaced)
+    (effects (font (size 1.27 1.27)) (justify right))
+    (property "Intersheetrefs" "${INTERSHEET_REFS}" (at 123.6104 91.44 0)
+      (effects (font (size 1.27 1.27)) (justify right) hide)
+    )
+  )
+  (global_label "SCL" (shape input) (at 135.89 104.14 180) (fields_autoplaced)
+    (effects (font (size 1.27 1.27)) (justify right))
+    (property "Intersheetrefs" "${INTERSHEET_REFS}" (at 129.4766 104.14 0)
+      (effects (font (size 1.27 1.27)) (justify right) hide)
+    )
+  )
+  (global_label "SDA" (shape input) (at 135.89 101.6 180) (fields_autoplaced)
+    (effects (font (size 1.27 1.27)) (justify right))
+    (property "Intersheetrefs" "${INTERSHEET_REFS}" (at 129.4161 101.6 0)
+      (effects (font (size 1.27 1.27)) (justify right) hide)
+    )
+  )
+  (symbol (lib_id "Connector_Generic:Conn_01x08") (at 143.51 93.98 0) (unit 1)
+    (in_bom yes) (on_board yes) (dnp no) (fields_autoplaced)
+    (property "Reference" "Camera" (at 146.05 94.615 0)
+      (effects (font (size 1.27 1.27)) (justify left))
+    )
+    (property "Value" "Conn_01x08" (at 146.05 97.155 0)
+      (effects (font (size 1.27 1.27)) (justify left))
+    )
+    (property "Footprint" "Connector_PinHeader_2.54mm:PinHeader_1x08_P2.54mm_Vertical" (at 143.51 93.98 0)
+      (effects (font (size 1.27 1.27)) hide)
+    )
+    (property "Datasheet" "~" (at 143.51 93.98 0)
+      (effects (font (size 1.27 1.27)) hide)
+    )
+    (pin "1")
+    (pin "2")
+    (pin "3")
+    (pin "4")
+    (pin "5")
+    (pin "6")
+    (pin "7")
+    (pin "8")
+    (instances
+      (project "Probe"
+        (path "/39298cfd-dda5-4ee5-9b0e-e5abd5a9144b/9a974da6-0248-442d-8149-85fb7bcb4159"
+          (reference "Camera") (unit 1)
+        )
+      )
+    )
+  )
+  (symbol (lib_id "power:GND") (at 135.89 96.52 270) (unit 1)
+    (in_bom yes) (on_board yes) (dnp no) (fields_autoplaced)
+    (property "Reference" "#PWR03" (at 129.54 96.52 0)
+      (effects (font (size 1.27 1.27)) hide)
+    )
+    (property "Value" "GND" (at 132.08 97.155 90)
+      (effects (font (size 1.27 1.27)) (justify right))
+    )
+    (property "Footprint" "" (at 135.89 96.52 0)
+      (effects (font (size 1.27 1.27)) hide)
+    )
+    (property "Datasheet" "" (at 135.89 96.52 0)
+      (effects (font (size 1.27 1.27)) hide)
+    )
+    (pin "1")
+    (instances
+      (project "Probe"
+        (path "/39298cfd-dda5-4ee5-9b0e-e5abd5a9144b/9a974da6-0248-442d-8149-85fb7bcb4159"
+          (reference "#PWR03") (unit 1)
+        )
+      )
+    )
+  )
 )
