File: HW/Controller.kicad_sch (KiCad schematic)
At the start: 0 parts

Commit message: Create probe pcb
Parts:
- added R1: R, symbol Device:R
- added U1: NUCLEO-L432KC, MODULE_NUCLEO-L432KC, symbol NUCLEO-L432KC:NUCLEO-L432KC
Connections:
- new net: R1.1, U1.CN4_14 (+3V3)
- new net: R1.2, U1.CN4_3 (NRST_CN4)
- new net 5V: U1.CN4_4 (+5V)
- new net CAM_CS: U1.CN3_6 (PB0)
- new net CAM_MISO: U1.CN4_7 (PA6)
- new net CAM_MOSI: U1.CN4_6 (PA7)
- new net CAM_SCK: U1.CN4_8 (PA5)
- new net GND: U1.CN3_4 (GND_CN3), U1.CN4_2 (GND_CN4)
- new net SCL: U1.CN3_1 (PA9)
- new net SDA: U1.CN3_2 (PA10)
- new net USB_DM: U1.CN3_13 (PA11)
- new net USB_DP: U1.CN3_5 (PA12)
